File: board-scope-R3.sch (EAGLE design)
At the start: 126 parts, among them IC3 STM32F103C8T, J2 12401598E4#2A, U1 HD3SS3220IRNHT, U2 TUSB8020B, U3 FT600Q-T, U4 ICE40HX1K-VQ100, U5 25F32006WSOI, U7 TPS54386, X1 30Mhz, X2 8Mhz, X3 24Mhz, Y1 OSCILLATORSMD-5X3

Commit message: done routing
Parts:
- R24: value (none) -> 10k
Connections:
- removed net BM_LED0-1: IC3MCU.PA9
- removed net BM_TDI: U$2.TDI
- removed net BM_TDO: U$2.TDO
- removed net FT_WAKE: U3.!WAKEUP
- removed net N$2: IC3MCU.PB9
- removed net N$56: U$1.B15
- removed net N$58: U$1.B7
- removed net N$6: U$2.RTCK
- removed net N$60: U$1.B14
- removed net N$65: U4.IOB_43_CBSEL1
- removed net N$8: IC3MCU.PB1
- removed net VUSB_3.0: R9.2
- net +3V3: now also R24.2, U2.VDD33
- net V_USB: now also R9.2
Changed lines of the file:
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@@
 </classes>
 <parts>
-<part name="FRAME1" library="frames" library_urn="urn:adsk.eagle:library:229" deviceset="A3L-LOC" device=""/>
+<part name="FRAME1" library="frames" library_urn="urn:adsk.eagle:library:229" deviceset="A3L-LOC" device="" value="test"/>
 <part name="FRAME2" library="frames" library_urn="urn:adsk.eagle:library:229" deviceset="A3L-LOC" device=""/>
 <part name="FRAME3" library="frames" library_urn="urn:adsk.eagle:library:229" deviceset="A3L-LOC" device=""/>
@@
 <part name="S2" library="mylib" deviceset="MOMENTARY-SWITCH-SPST-2" device="-SMD-5.2MM"/>
 <part name="SUPPLY51" library="supply2" library_urn="urn:adsk.eagle:library:372" deviceset="GND" device=""/>
-<part name="R24" library="rcl" library_urn="urn:adsk.eagle:library:334" deviceset="R-US_" device="R0603" package3d_urn="urn:adsk.eagle:package:23555/2"/>
+<part name="R24" library="rcl" library_urn="urn:adsk.eagle:library:334" deviceset="R-US_" device="R0603" package3d_urn="urn:adsk.eagle:package:23555/2" value="10k"/>
 <part name="+3V18" library="supply1" deviceset="+3V3" device=""/>
 <part name="R25" library="rcl" library_urn="urn:adsk.eagle:library:334" deviceset="R-US_" device="R0603" package3d_urn="urn:adsk.eagle:package:23555/2" value="10k"/>
@@
 <part name="SUPPLY56" library="supply2" library_urn="urn:adsk.eagle:library:372" deviceset="GND" device=""/>
 <part name="SUPPLY57" library="supply2" library_urn="urn:adsk.eagle:library:372" deviceset="GND" device=""/>
+<part name="SUPPLY33" library="SparkFun-PowerSymbols" library_urn="urn:adsk.eagle:library:530" deviceset="V_USB" device=""/>
 </parts>
 <sheets>
@@
 </segment>
 </net>
-<net name="BM_TDO" class="0">
-<segment>
-<pinref part="U$2" gate="G$1" pin="TDO"/>
-<wire x1="350.52" y1="218.44" x2="340.36" y2="218.44" width="0.1524" layer="91"/>
-<label x="340.36" y="218.44" size="1.778" layer="95"/>
-</segment>
-</net>
 <net name="BM_TMS" class="0">
 <segment>
@@
 </segment>
 </net>
-<net name="BM_TDI" class="0">
-<segment>
-<pinref part="U$2" gate="G$1" pin="TDI"/>
-<wire x1="350.52" y1="238.76" x2="340.36" y2="238.76" width="0.1524" layer="91"/>
-<label x="340.36" y="238.76" size="1.778" layer="95"/>
-</segment>
-</net>
 <net name="BM_TRGT_SWDIO_IN" class="0">
 <segment>
@@
 </segment>
 </net>
-<net name="N$8" class="0">
-<segment>
-<pinref part="IC3" gate="MCU" pin="PB1"/>
-<wire x1="132.08" y1="162.56" x2="152.4" y2="162.56" width="0.1524" layer="91"/>
-</segment>
-</net>
 <net name="BM_TX" class="0">
 <segment>
@@
 </segment>
 </net>
-<net name="BM_LED0-1" class="0">
-<segment>
-<pinref part="IC3" gate="MCU" pin="PA9"/>
-<wire x1="132.08" y1="139.7" x2="148.59" y2="139.7" width="0.1524" layer="91"/>
-<label x="134.62" y="139.7" size="1.778" layer="95"/>
-</segment>
-</net>
 <net name="N$16" class="0">
 <segment>
@@
 </segment>
 </net>
-<net name="N$6" class="0">
-<segment>
-<pinref part="U$2" gate="G$1" pin="RTCK"/>
-<wire x1="350.52" y1="203.2" x2="340.36" y2="203.2" width="0.1524" layer="91"/>
-</segment>
-</net>
 <net name="BM_SCK" class="0">
 <segment>
@@
 </segment>
 </net>
-<net name="N$2" class="0">
-<segment>
-<pinref part="IC3" gate="MCU" pin="PB9"/>
-<wire x1="132.08" y1="182.88" x2="152.4" y2="182.88" width="0.1524" layer="91"/>
-</segment>
-</net>
 <net name="N$3" class="0">
 <segment>
@@
 <instance part="C655" gate="G$1" x="76.2" y="46.99"/>
 <instance part="C656" gate="G$1" x="86.36" y="46.99"/>
-<instance part="VCC1" gate="G$1" x="17.78" y="57.15"/>
+<instance part="VCC1" gate="G$1" x="17.78" y="59.69"/>
 <instance part="VCC3" gate="G$1" x="167.64" y="207.01"/>
 <instance part="D4" gate="G$1" x="177.8" y="184.15" rot="R180"/>
@@
 <segment>
 <pinref part="C650" gate="G$1" pin="1"/>
-<wire x1="17.78" y1="54.61" x2="17.78" y2="52.07" width="0.1524" layer="91"/>
+<wire x1="17.78" y1="57.15" x2="17.78" y2="52.07" width="0.1524" layer="91"/>
 <pinref part="C651" gate="G$1" pin="1"/>
 <wire x1="17.78" y1="52.07" x2="17.78" y2="49.53" width="0.1524" layer="91"/>
@@
 <wire x1="86.36" y1="52.07" x2="86.36" y2="49.53" width="0.1524" layer="91"/>
 <junction x="76.2" y="52.07"/>
+<pinref part="VCC1" gate="G$1" pin="VCCINT"/>
 </segment>
 </net>
@@
 <wire x1="350.52" y1="179.07" x2="350.52" y2="186.69" width="0.1524" layer="91"/>
 </segment>
+<segment>
+<pinref part="R24" gate="G$1" pin="2"/>
+<pinref part="+3V18" gate="G$1" pin="+3V3"/>
+<wire x1="255.27" y1="105.41" x2="255.27" y2="106.68" width="0.1524" layer="91"/>
+</segment>
 </net>
 <net name="N$1" class="0">
@@
 </segment>
 </net>
-<net name="N$65" class="0">
-<segment>
-<pinref part="U4" gate="G$1" pin="IOB_43_CBSEL1"/>
-<wire x1="106.68" y1="90.17" x2="92.71" y2="90.17" width="0.1524" layer="91"/>
-</segment>
-</net>
 </nets>
 </sheet>
@@
 <text x="312.42" y="144.78" size="1.778" layer="94">x</text>
 <text x="312.42" y="147.32" size="1.778" layer="94">x</text>
+<text x="203.2" y="187.96" size="1.778" layer="94">x</text>
+<text x="203.2" y="185.42" size="1.778" layer="94">x</text>
 </plain>
 <instances>
@@
 <wire x1="248.92" y1="68.58" x2="243.84" y2="68.58" width="0.1524" layer="91"/>
 <junction x="243.84" y="68.58"/>
+<pinref part="U2" gate="G$1" pin="VDD33"/>
 <wire x1="248.92" y1="71.12" x2="243.84" y2="71.12" width="0.1524" layer="91"/>
 <junction x="243.84" y="71.12"/>
@@
 <instance part="R26" gate="G$1" x="45.72" y="142.24" rot="R90"/>
 <instance part="+3V21" gate="G$1" x="45.72" y="151.13"/>
+<instance part="SUPPLY33" gate="G$1" x="227.33" y="165.1"/>
 </instances>
 <busses>
@@
 </segment>
 </net>
-<net name="VUSB_3.0" class="0">
-<segment>
-<pinref part="R9" gate="G$1" pin="2"/>
-<wire x1="227.33" y1="158.75" x2="227.33" y2="163.83" width="0.1524" layer="91"/>
-<wire x1="227.33" y1="163.83" x2="240.03" y2="163.83" width="0.1524" layer="91"/>
-<label x="229.87" y="163.83" size="1.778" layer="95"/>
-</segment>
-</net>
 <net name="FT_SIWU" class="0">
 <segment>
@@
 </segment>
 </net>
-<net name="FT_WAKE" class="0">
-<segment>
-<pinref part="U3" gate="G$1" pin="!WAKEUP"/>
-<wire x1="87.63" y1="129.54" x2="63.5" y2="129.54" width="0.1524" layer="91"/>
-<label x="66.04" y="129.54" size="1.778" layer="95"/>
-</segment>
-</net>
 <net name="FT_VUSB_DET" class="0">
 <segment>
@@
 </segment>
 </net>
+<net name="V_USB" class="0">
+<segment>
+<pinref part="R9" gate="G$1" pin="2"/>
+<wire x1="227.33" y1="158.75" x2="227.33" y2="165.1" width="0.1524" layer="91"/>
+<pinref part="SUPPLY33" gate="G$1" pin="V_USB"/>
+</segment>
+</net>
 </nets>
 </sheet>
@@
 </segment>
 </net>
-<net name="N$58" class="0">
-<segment>
-<pinref part="U$1" gate="G$1" pin="B7"/>
-<wire x1="325.12" y1="91.44" x2="345.44" y2="91.44" width="0.1524" layer="91"/>
-</segment>
-</net>
 <net name="ICE_CRESET" class="0">
 <segment>
@@
 </segment>
 </net>
-<net name="N$56" class="0">
-<segment>
-<pinref part="U$1" gate="G$1" pin="B15"/>
-<wire x1="276.86" y1="86.36" x2="287.02" y2="86.36" width="0.1524" layer="91"/>
-</segment>
-</net>
-<net name="N$60" class="0">
-<segment>
-<pinref part="U$1" gate="G$1" pin="B14"/>
-<wire x1="276.86" y1="91.44" x2="287.02" y2="91.44" width="0.1524" layer="91"/>
-</segment>
-</net>
 <net name="ICE_SS" class="0">
 <segment>
@@
 </sheet>
 </sheets>
+<errors>
+</errors>
 </schematic>
 </drawing>
